Commit message: updates

File: src/yahboomcar_description/urdf/yahboomcar_X3.urdf (robot description, URDF)
Before this commit: robot yahboomcar, 9 links, 8 joints
Joints:
- joint laser_joint: origin xyz=0.0435 5.25826986680105E-05 0.11 rpy=0 0 0 -> xyz=0.0435 5.25826986680105E-05 0.11 rpy=0 0 3.14159265

File: src/yahboomcar_description/urdf/yahboomcar_X3.urdf.xacro (robot description, xacro)
@@ -110,5 +110,5 @@
         </inertial>
     </common_link>
-    <fixed_joint name="laser_joint" parent="base_link" child="laser_link" xyz="0.0435 5.25826986680105E-05 0.11" rpy="0 0 0"/>
+    <fixed_joint name="laser_joint" parent="base_link" child="laser_link" xyz="0.0435 5.25826986680105E-05 0.11" rpy="0 0 3.14159265"/>
     <common_link name="camera_link" material="White" path="sensor">
         <inertial>
