Commit message: updates

File: src/yahboomcar_description/urdf/yahboomcar_X3.urdf (robot description, URDF)
Before this commit: robot yahboomcar, 9 links, 8 joints
Links:
- added link lidar_mount_link, mass 0.035; collision mesh filename=package://yahboomcar_description/meshes/4ROS_lidar_mount.STL scale=0.001 0.001 0.001; visual mesh filename=package://yahboomcar_description/meshes/4ROS_lidar_mount.STL scale=0.001 0.001 0.001
Joints:
- added joint lidar_mount_joint: type fixed, parent base_link, child lidar_mount_link, origin xyz=0.0435 5.25826986680105E-05 0.11 rpy=0 0 0
- joint laser_joint: origin xyz=0.0435 5.25826986680105E-05 0.11 rpy=0 0 3.14159265 -> xyz=0.0435 5.25826986680105E-05 0.185 rpy=0 0 3.14159265

File: src/yahboomcar_description/urdf/yahboomcar_X3.urdf.xacro (robot description, xacro)
@@ -110,5 +110,27 @@
         </inertial>
     </common_link>
-    <fixed_joint name="laser_joint" parent="base_link" child="laser_link" xyz="0.0435 5.25826986680105E-05 0.11" rpy="0 0 3.14159265"/>
+    <link name="${ns}/lidar_mount_link">
+        <inertial>
+            <origin xyz="0 0 0.0375" rpy="0 0 0"/>
+            <mass value="0.035"/>
+            <inertia ixx="2.55E-05" ixy="0" ixz="0"
+                     iyy="2.55E-05" iyz="0" izz="1.76E-05"/>
+        </inertial>
+        <visual>
+            <origin xyz="-0.0275 0.03368 0" rpy="1.5707963 0 0"/>
+            <geometry>
+                <mesh filename="package://yahboomcar_description/meshes/4ROS_lidar_mount.STL" scale="0.001 0.001 0.001"/>
+            </geometry>
+            <material name="White"/>
+        </visual>
+        <collision>
+            <origin xyz="-0.0275 0.03368 0" rpy="1.5707963 0 0"/>
+            <geometry>
+                <mesh filename="package://yahboomcar_description/meshes/4ROS_lidar_mount.STL" scale="0.001 0.001 0.001"/>
+            </geometry>
+        </collision>
+    </link>
+    <fixed_joint name="lidar_mount_joint" parent="base_link" child="lidar_mount_link" xyz="0.0435 5.25826986680105E-05 0.11" rpy="0 0 0"/>
+    <fixed_joint name="laser_joint" parent="base_link" child="laser_link" xyz="0.0435 5.25826986680105E-05 0.185" rpy="0 0 3.14159265"/>
     <common_link name="camera_link" material="White" path="sensor">
         <inertial>

Commit message: chore: update robot meshes, YOLO model artifacts, navigation configuration, and build scripts across multiple worktrees.

File: src/yahboomcar_description/urdf/yahboomcar_X3.urdf (robot description, URDF)
Before this commit: robot yahboomcar, 10 links, 9 joints
Links:
- added link oak-d-base-frame, mass 0.0611; collision box size=0.028 0.091 0.0175; visual box size=0.028 0.091 0.0175
- added link oak_imu_frame
- added link oak_left_camera_frame
- added link oak_left_camera_optical_frame
- added link oak_rgb_camera_frame
- added link oak_rgb_camera_optical_frame
- added link oak_right_camera_frame
- added link oak_right_camera_optical_frame
Joints:
- added joint oak_center_joint: type fixed, parent base_link, child oak-d-base-frame, origin xyz=0.0435 5.25826986680105E-05 0.185 rpy=0 0 0
- added joint oak_imu_joint: type fixed, parent oak-d-base-frame, child oak_imu_frame, origin xyz=0 0 0 rpy=0 0 0
- added joint oak_left_camera_joint: type fixed, parent oak-d-base-frame, child oak_left_camera_frame, origin xyz=0 0.0375 0 rpy=0 0 0
- added joint oak_left_camera_optical_joint: type fixed, parent oak_left_camera_frame, child oak_left_camera_optical_frame, origin xyz=0 0 0 rpy=-1.5707963 0 -1.5707963
- added joint oak_rgb_camera_joint: type fixed, parent oak-d-base-frame, child oak_rgb_camera_frame, origin xyz=0 0 0 rpy=0 0 0
- added joint oak_rgb_camera_optical_joint: type fixed, parent oak_rgb_camera_frame, child oak_rgb_camera_optical_frame, origin xyz=0 0 0 rpy=-1.5707963 0 -1.5707963
- added joint oak_right_camera_joint: type fixed, parent oak-d-base-frame, child oak_right_camera_frame, origin xyz=0 -0.0375 0 rpy=0 0 0
- added joint oak_right_camera_optical_joint: type fixed, parent oak_right_camera_frame, child oak_right_camera_optical_frame, origin xyz=0 0 0 rpy=-1.5707963 0 -1.5707963
- joint laser_joint: origin xyz=0.0435 5.25826986680105E-05 0.185 rpy=0 0 3.14159265 -> xyz=-0.0115 5.25826986680105E-05 0.191 rpy=0 0 3.14159265
- joint lidar_mount_joint: origin xyz=0.0435 5.25826986680105E-05 0.11 rpy=0 0 0 -> xyz=-0.0115 5.25826986680105E-05 0.116 rpy=0 0 0

File: src/yahboomcar_description/urdf/yahboomcar_X3.urdf.xacro (robot description, xacro)
@@ -131,6 +131,7 @@
         </collision>
     </link>
-    <fixed_joint name="lidar_mount_joint" parent="base_link" child="lidar_mount_link" xyz="0.0435 5.25826986680105E-05 0.11" rpy="0 0 0"/>
-    <fixed_joint name="laser_joint" parent="base_link" child="laser_link" xyz="0.0435 5.25826986680105E-05 0.185" rpy="0 0 3.14159265"/>
+    <!-- lidar moved 55 mm rearward, 6 mm up (2026); OAK-D took its old front spot -->
+    <fixed_joint name="lidar_mount_joint" parent="base_link" child="lidar_mount_link" xyz="-0.0115 5.25826986680105E-05 0.116" rpy="0 0 0"/>
+    <fixed_joint name="laser_joint" parent="base_link" child="laser_link" xyz="-0.0115 5.25826986680105E-05 0.191" rpy="0 0 3.14159265"/>
     <common_link name="camera_link" material="White" path="sensor">
         <inertial>
@@ -141,3 +142,47 @@
     </common_link>
     <fixed_joint name="camera_joint" parent="base_link" child="camera_link" xyz="0.057105 1.7948E-05 0.03755" rpy="0 0 0"/>
+    <!-- ==================== OAK-D Lite (2026) ====================
+         Mounted at the lidar's previous front location (x=0.0435, z=0.185).
+         Frame names follow the depthai_ros convention (camera name "oak").
+         Stereo baseline 75 mm: left mono +Y, right mono -Y. -->
+    <link name="${ns}/oak-d-base-frame">
+        <inertial>
+            <origin xyz="0 0 0" rpy="0 0 0"/>
+            <mass value="0.0611"/>
+            <inertia ixx="4.3E-05" ixy="0" ixz="0"
+                     iyy="4.5E-06" iyz="0" izz="4.5E-05"/>
+        </inertial>
+        <visual>
+            <origin xyz="0 0 0" rpy="0 0 0"/>
+            <geometry>
+                <box size="0.028 0.091 0.0175"/>
+            </geometry>
+            <material name="White"/>
+        </visual>
+        <collision>
+            <origin xyz="0 0 0" rpy="0 0 0"/>
+            <geometry>
+                <box size="0.028 0.091 0.0175"/>
+            </geometry>
+        </collision>
+    </link>
+    <fixed_joint name="oak_center_joint" parent="base_link" child="oak-d-base-frame" xyz="0.0435 5.25826986680105E-05 0.185" rpy="0 0 0"/>
+    <!-- RGB camera (center) -->
+    <link name="${ns}/oak_rgb_camera_frame"/>
+    <fixed_joint name="oak_rgb_camera_joint" parent="oak-d-base-frame" child="oak_rgb_camera_frame" xyz="0 0 0" rpy="0 0 0"/>
+    <link name="${ns}/oak_rgb_camera_optical_frame"/>
+    <fixed_joint name="oak_rgb_camera_optical_joint" parent="oak_rgb_camera_frame" child="oak_rgb_camera_optical_frame" xyz="0 0 0" rpy="${-pi/2} 0 ${-pi/2}"/>
+    <!-- Left mono camera (+Y) -->
+    <link name="${ns}/oak_left_camera_frame"/>
+    <fixed_joint name="oak_left_camera_joint" parent="oak-d-base-frame" child="oak_left_camera_frame" xyz="0 0.0375 0" rpy="0 0 0"/>
+    <link name="${ns}/oak_left_camera_optical_frame"/>
+    <fixed_joint name="oak_left_camera_optical_joint" parent="oak_left_camera_frame" child="oak_left_camera_optical_frame" xyz="0 0 0" rpy="${-pi/2} 0 ${-pi/2}"/>
+    <!-- Right mono camera (-Y) -->
+    <link name="${ns}/oak_right_camera_frame"/>
+    <fixed_joint name="oak_right_camera_joint" parent="oak-d-base-frame" child="oak_right_camera_frame" xyz="0 -0.0375 0" rpy="0 0 0"/>
+    <link name="${ns}/oak_right_camera_optical_frame"/>
+    <fixed_joint name="oak_right_camera_optical_joint" parent="oak_right_camera_frame" child="oak_right_camera_optical_frame" xyz="0 0 0" rpy="${-pi/2} 0 ${-pi/2}"/>
+    <!-- On-board IMU -->
+    <link name="${ns}/oak_imu_frame"/>
+    <fixed_joint name="oak_imu_joint" parent="oak-d-base-frame" child="oak_imu_frame" xyz="0 0 0" rpy="0 0 0"/>
 </robot>

Commit message: feat(urdf): establish X3 Plus geometry baseline

File: src/yahboomcar_description/urdf/yahboomcar_X3.urdf (robot description, URDF)
Before this commit: robot yahboomcar, 20 links, 19 joints
Links:
- link base_link: mass 0.486218814966626 -> 1.0754239466482; geometry collision mesh filename=package://yahboomcar_description/meshes/X3plus/collision/ba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; visual mesh filename=package://yahboomcar_description/meshes/X3plus/visual/base_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
Joints:
- joint base_joint: origin xyz=0.0 0.0 0.0815 rpy=0 0 0 -> xyz=0.0 0.0 0.076 rpy=0 0 0
- joint oak_center_joint: origin xyz=0.0435 5.25826986680105E-05 0.185 rpy=0 0 0 -> xyz=0.0435 5.25826986680105E-05 0.134 rpy=0 0 0

Commit message: fix(urdf): remove duplicate X3 wheel meshes

File: src/yahboomcar_description/urdf/yahboomcar_X3.urdf (robot description, URDF)
Before this commit: robot yahboomcar, 20 links, 19 joints
Links:
- link back_left_wheel: mass 0.0515309299357028 -> None; geometry 
- link back_right_wheel: mass 0.051540174053366 -> None; geometry 
- link front_left_wheel: mass 0.051543 -> None; geometry 
- link front_right_wheel: mass 0.051532 -> None; geometry 

Commit message: fix(urdf): place Astra 18 mm behind X3 Plus front

File: src/yahboomcar_description/urdf/yahboomcar_X3.urdf (robot description, URDF)
Before this commit: robot yahboomcar, 20 links, 19 joints
Joints:
- joint camera_joint: origin xyz=0.057105 1.7948E-05 0.03755 rpy=0 0 0 -> xyz=0.107315 1.7948E-05 0.03755 rpy=0 0 0

Commit message: fix(urdf): align OAK-D directly above Astra

File: src/yahboomcar_description/urdf/yahboomcar_X3.urdf (robot description, URDF)
Before this commit: robot yahboomcar, 20 links, 19 joints
Joints:
- joint oak_center_joint: origin xyz=0.0435 5.25826986680105E-05 0.134 rpy=0 0 0 -> xyz=0.107315 1.7948E-05 0.134 rpy=0 0 0

Commit message: fix(urdf): seat lidar mount and ICM on top plate

File: src/yahboomcar_description/urdf/yahboomcar_X3.urdf (robot description, URDF)
Before this commit: robot yahboomcar, 20 links, 19 joints
Joints:
- joint base_icm_imu: origin xyz=-0.03 0 0.0885 rpy=0 0 0 -> xyz=-0.03 0 0.062 rpy=0 0 0
- joint lidar_mount_joint: origin xyz=0.0557 5.25826986680105E-05 0.0885 rpy=0 0 0 -> xyz=0.0557 5.25826986680105E-05 0.062 rpy=0 0 0

Commit message: feat(urdf): add measured 12 V battery envelope

File: src/yahboomcar_description/urdf/yahboomcar_X3.urdf (robot description, URDF)
Before this commit: robot yahboomcar, 20 links, 19 joints
Links:
- added link battery_link; collision box size=0.061 0.114 0.075; visual box size=0.061 0.114 0.075
Joints:
- added joint battery_joint: type fixed, parent base_link, child battery_link, origin xyz=-0.096 0 0.062 rpy=0 0 0

Commit message: fix(urdf): move battery 5 mm forward

File: src/yahboomcar_description/urdf/yahboomcar_X3.urdf (robot description, URDF)
Before this commit: robot yahboomcar, 21 links, 20 joints
Joints:
- joint battery_joint: origin xyz=-0.096 0 0.062 rpy=0 0 0 -> xyz=-0.091 0 0.062 rpy=0 0 0
