Commit message: Model dual ToF mount at confirmed chassis placement

File: src/yahboomcar_description/urdf/yahboomcar_X3.urdf (robot description, URDF)
Before this commit: robot yahboomcar, 26 links, 25 joints
Links:
- added link tof_lower_board_link; collision mesh filename=package://yahboomcar_description/meshes/tof_breakout.stl; visual mesh filename=package://yahboomcar_description/meshes/tof_breakout.stl
- added link tof_lower_link
- added link tof_lower_optical_frame
- added link tof_upper_board_link; collision mesh filename=package://yahboomcar_description/meshes/tof_breakout.stl; visual mesh filename=package://yahboomcar_description/meshes/tof_breakout.stl
- added link tof_upper_link
- added link tof_upper_optical_frame
- link tof_mount_link: mass 0.030 -> None; geometry collision mesh filename=package://yahboomcar_description/meshes/tof_adapter_15.stl; collision mesh filename=package://yahboomcar_description/meshes/tof_adapter_40.stl
Joints:
- added joint tof_lower_board_joint: type fixed, parent tof_mount_link, child tof_lower_board_link, origin xyz=-0.000100000 0.018035352 0.019528620 rpy=-2.443460930 -0.000000000 -0.000000000
- added joint tof_lower_joint: type fixed, parent tof_mount_link, child tof_lower_link, origin xyz=-0.000100000 0.014892252 0.019462898 rpy=0.000000000 -0.872664626 -1.570796327
- added joint tof_lower_optical_joint: type fixed, parent tof_lower_link, child tof_lower_optical_frame, origin xyz=0 0 0 rpy=-1.570796326795 0 -1.570796326795
- added joint tof_upper_board_joint: type fixed, parent tof_mount_link, child tof_upper_board_link, origin xyz=-0.000100000 0.113745168 0.016700834 rpy=-2.879793264 -0.000000000 0.000000000
- added joint tof_upper_joint: type fixed, parent tof_mount_link, child tof_upper_link, origin xyz=-0.000100000 0.110868776 0.017969601 rpy=0.000000000 -1.308996939 -1.570796327
- added joint tof_upper_optical_joint: type fixed, parent tof_upper_link, child tof_upper_optical_frame, origin xyz=0 0 0 rpy=-1.570796326795 0 -1.570796326795
- joint tof_joint: origin xyz=0.000115 0.016049 0.017941 rpy=0 -1.3089969 -1.5707963 -> xyz=0 0 0 rpy=0 0 0; parent tof_mount_link -> tof_upper_link
- joint tof_mount_joint: origin xyz=0.1320 0.0 -0.033549 rpy=1.5707963 0 1.5707963 -> xyz=0.1450 0.0 -0.030549 rpy=1.570796326795 0 1.570796326795
- joint tof_optical_joint: origin xyz=0 0 0 rpy=-1.5707963 0 -1.5707963 -> xyz=0 0 0 rpy=-1.570796326795 0 -1.570796326795

File: src/yahboomcar_description/urdf/yahboomcar_X3.urdf.xacro (robot description, xacro)
@@ -11,9 +11,9 @@
     <link name="${ns}/imu_link"/>
     <!-- common link-->
-    <xacro:macro name="common_link" params="name material path *origin">
+    <xacro:macro name="common_link" params="name material path *origin mesh_suffix:=''">
         <link name="${ns}/${name}">
             <visual>
                 <geometry>
-                    <mesh filename="package://yahboomcar_description/meshes/${path}/${name}.STL"/>
+                    <mesh filename="package://yahboomcar_description/meshes/${path}/${name}${mesh_suffix}.STL"/>
                 </geometry>
                 <origin xyz="0 0 0" rpy="0 0 0"/>
@@ -22,5 +22,5 @@
             <collision>
                 <geometry>
-                    <mesh filename="package://yahboomcar_description/meshes/${path}/${name}.STL"/>
+                    <mesh filename="package://yahboomcar_description/meshes/${path}/${name}${mesh_suffix}.STL"/>
                 </geometry>
                 <origin xyz="0 0 0" rpy="0 0 0"/>
@@ -47,5 +47,5 @@
         </joint>
     </xacro:macro>
-    <common_link name="base_link" material="Green" path="mecanum">
+    <xacro:common_link name="base_link" material="Green" path="mecanum" mesh_suffix="_X3">
         <inertial>
             <origin xyz="0.00498197982182523 5.70233829969297E-05 -0.0121008098068578" rpy="0 0 0"/>
@@ -59,8 +59,8 @@
                     izz="0.00493927269870476"/>
         </inertial>
-    </common_link>
-    <fixed_joint name="base_joint" parent="base_footprint" child="base_link" xyz="0.0 0.0 0.0815" rpy="0 0 0"/>
-    <fixed_joint name="base_imu" parent="base_link" child="imu_link" xyz="-0.06 0.01 0.01" rpy="0 3.1415 1.5707"/>
-    <common_link name="front_right_wheel" material="White" path="mecanum">
+    </xacro:common_link>
+    <xacro:fixed_joint name="base_joint" parent="base_footprint" child="base_link" xyz="0.0 0.0 0.0815" rpy="0 0 0"/>
+    <xacro:fixed_joint name="base_imu" parent="base_link" child="imu_link" xyz="-0.06 0.01 0.01" rpy="0 3.1415 1.5707"/>
+    <xacro:common_link name="front_right_wheel" material="White" path="mecanum" mesh_suffix="_X3">
         <inertial>
             <origin xyz="1.9051E-06 -2.3183E-07 -0.00064079" rpy="0 0 0"/>
@@ -69,8 +69,8 @@
                      iyy="1.4594E-05" iyz="-1.7476E-09" izz="2.4264E-05"/>
         </inertial>
-    </common_link>
-    <continuous_joint name="front_right_joint" parent="base_link" child="front_right_wheel"
+    </xacro:common_link>
+    <xacro:continuous_joint name="front_right_joint" parent="base_link" child="front_right_wheel"
                       xyz="0.08 -0.0845 -0.0389" rpy="-${pi/2} 0 ${pi}" axis="0 0 1"/>
-    <common_link name="front_left_wheel" material="White" path="mecanum">
+    <xacro:common_link name="front_left_wheel" material="White" path="mecanum" mesh_suffix="_X3">
         <inertial>
             <origin xyz="2.3728E-06 -9.4228E-07 0.00064068" rpy="0 0 0"/>
@@ -79,8 +79,8 @@
                      iyy="1.4598E-05" iyz="1.7972E-09" izz="2.4267E-05"/>
         </inertial>
-    </common_link>
-    <continuous_joint name="front_left_joint" parent="base_link" child="front_left_wheel"
+    </xacro:common_link>
+    <xacro:continuous_joint name="front_left_joint" parent="base_link" child="front_left_wheel"
                       xyz="0.08 0.084492 -0.0389" rpy="${pi/2} 0 0" axis="0 0 1"/>
-    <common_link name="back_right_wheel" material="White" path="mecanum">
+    <xacro:common_link name="back_right_wheel" material="White" path="mecanum" mesh_suffix="_X3">
         <inertial>
             <origin xyz="-1.75924169923403E-06 1.28388821071107E-06 -0.000590549296238266" rpy="0 0 0"/>
@@ -89,8 +89,8 @@
                      iyy="1.4596501955693E-05" iyz="-6.27904057423818E-10" izz="2.42663091380451E-05"/>
         </inertial>
-    </common_link>
-    <continuous_joint name="back_right_joint" parent="base_link" child="back_right_wheel"
+    </xacro:common_link>
+    <xacro:continuous_joint name="back_right_joint" parent="base_link" child="back_right_wheel"
                       xyz="-0.08 -0.0845 -0.03946" rpy="-${pi/2} 0 ${pi}" axis="0 0 1"/>
-    <common_link name="back_left_wheel" material="White" path="mecanum">
+    <xacro:common_link name="back_left_wheel" material="White" path="mecanum" mesh_suffix="_X3">
         <inertial>
             <origin xyz="-4.01213085227115E-07 2.04910264598596E-06 0.000590775697051377" rpy="0 0 0"/>
@@ -99,8 +99,8 @@
                      iyy="1.45948727598913E-05" iyz="1.61769812110049E-10" izz="2.4263683888153E-05"/>
         </inertial>
-    </common_link>
-    <continuous_joint name="back_left_joint" parent="base_link" child="back_left_wheel"
+    </xacro:common_link>
+    <xacro:continuous_joint name="back_left_joint" parent="base_link" child="back_left_wheel"
                       xyz="-0.08 0.084492 -0.03954" rpy="${pi/2} 0 0" axis="0 0 1"/>
-    <common_link name="laser_link" material="White" path="sensor">
+    <xacro:common_link name="laser_link" material="White" path="sensor">
         <inertial>
             <origin xyz="-0.0176558922685589 0.000671805271544437 0.0219302095894866" rpy="0 0 0"/>
@@ -109,5 +109,5 @@
                      iyy="3.89262522903605E-05" iyz="3.24809725932687E-07" izz="4.86230801106223E-05"/>
         </inertial>
-    </common_link>
+    </xacro:common_link>
     <!-- ============ 2D->3D tilting lidar mount (2026-08) ============
          Bottom plate + 4ROS adapter bolt to the chassis; the lidar rides in a
@@ -169,5 +169,5 @@
         <xacro:mount_bearing xyz="-0.026141 -0.034900 0.145522" rpy="1.5707963 0.2839484 0"/>
     </link>
-    <fixed_joint name="lidar_mount_joint" parent="base_link" child="lidar_mount_link" xyz="0.0557 5.25826986680105E-05 0.0885" rpy="0 0 0"/>
+    <xacro:fixed_joint name="lidar_mount_joint" parent="base_link" child="lidar_mount_link" xyz="0.0557 5.25826986680105E-05 0.0885" rpy="0 0 0"/>
     <!-- Rotating cradle: carousel + shaft coupler -->
     <link name="${ns}/lidar_tilt_link">
@@ -197,6 +197,6 @@
         <limit lower="-2.0944" upper="2.0944" effort="1.6" velocity="6.5"/>
     </joint>
-    <fixed_joint name="laser_joint" parent="lidar_tilt_link" child="laser_link" xyz="0 0 0.022" rpy="0 0 3.14159265"/>
-    <common_link name="camera_link" material="White" path="sensor">
+    <xacro:fixed_joint name="laser_joint" parent="lidar_tilt_link" child="laser_link" xyz="0 0 0.022" rpy="0 0 3.14159265"/>
+    <xacro:common_link name="camera_link" material="White" path="sensor">
         <inertial>
             <origin xyz="0 0 0" rpy="0 0 0"/>
@@ -204,6 +204,6 @@
             <inertia ixx="0" ixy="0" ixz="0" iyy="0" iyz="0" izz="0"/>
         </inertial>
-    </common_link>
-    <fixed_joint name="camera_joint" parent="base_link" child="camera_link" xyz="0.057105 1.7948E-05 0.03755" rpy="0 0 0"/>
+    </xacro:common_link>
+    <xacro:fixed_joint name="camera_joint" parent="base_link" child="camera_link" xyz="0.057105 1.7948E-05 0.03755" rpy="0 0 0"/>
     <!-- ==================== OAK-D Lite (2026) ====================
          Mounted at the lidar's previous front location (x=0.0435, z=0.185).
@@ -231,76 +231,105 @@
         </collision>
     </link>
-    <fixed_joint name="oak_center_joint" parent="base_link" child="oak-d-base-frame" xyz="0.0435 5.25826986680105E-05 0.185" rpy="0 0 0"/>
+    <xacro:fixed_joint name="oak_center_joint" parent="base_link" child="oak-d-base-frame" xyz="0.0435 5.25826986680105E-05 0.185" rpy="0 0 0"/>
     <!-- RGB camera (center) -->
     <link name="${ns}/oak_rgb_camera_frame"/>
-    <fixed_joint name="oak_rgb_camera_joint" parent="oak-d-base-frame" child="oak_rgb_camera_frame" xyz="0 0 0" rpy="0 0 0"/>
+    <xacro:fixed_joint name="oak_rgb_camera_joint" parent="oak-d-base-frame" child="oak_rgb_camera_frame" xyz="0 0 0" rpy="0 0 0"/>
     <link name="${ns}/oak_rgb_camera_optical_frame"/>
-    <fixed_joint name="oak_rgb_camera_optical_joint" parent="oak_rgb_camera_frame" child="oak_rgb_camera_optical_frame" xyz="0 0 0" rpy="${-pi/2} 0 ${-pi/2}"/>
+    <xacro:fixed_joint name="oak_rgb_camera_optical_joint" parent="oak_rgb_camera_frame" child="oak_rgb_camera_optical_frame" xyz="0 0 0" rpy="${-pi/2} 0 ${-pi/2}"/>
     <!-- Left mono camera (+Y) -->
     <link name="${ns}/oak_left_camera_frame"/>
-    <fixed_joint name="oak_left_camera_joint" parent="oak-d-base-frame" child="oak_left_camera_frame" xyz="0 0.0375 0" rpy="0 0 0"/>
+    <xacro:fixed_joint name="oak_left_camera_joint" parent="oak-d-base-frame" child="oak_left_camera_frame" xyz="0 0.0375 0" rpy="0 0 0"/>
     <link name="${ns}/oak_left_camera_optical_frame"/>
-    <fixed_joint name="oak_left_camera_optical_joint" parent="oak_left_camera_frame" child="oak_left_camera_optical_frame" xyz="0 0 0" rpy="${-pi/2} 0 ${-pi/2}"/>
+    <xacro:fixed_joint name="oak_left_camera_optical_joint" parent="oak_left_camera_frame" child="oak_left_camera_optical_frame" xyz="0 0 0" rpy="${-pi/2} 0 ${-pi/2}"/>
     <!-- Right mono camera (-Y) -->
     <link name="${ns}/oak_right_camera_frame"/>
-    <fixed_joint name="oak_right_camera_joint" parent="oak-d-base-frame" child="oak_right_camera_frame" xyz="0 -0.0375 0" rpy="0 0 0"/>
+    <xacro:fixed_joint name="oak_right_camera_joint" parent="oak-d-base-frame" child="oak_right_camera_frame" xyz="0 -0.0375 0" rpy="0 0 0"/>
     <link name="${ns}/oak_right_camera_optical_frame"/>
-    <fixed_joint name="oak_right_camera_optical_joint" parent="oak_right_camera_frame" child="oak_right_camera_optical_frame" xyz="0 0 0" rpy="${-pi/2} 0 ${-pi/2}"/>
+    <xacro:fixed_joint name="oak_right_camera_optical_joint" parent="oak_right_camera_frame" child="oak_right_camera_optical_frame" xyz="0 0 0" rpy="${-pi/2} 0 ${-pi/2}"/>
     <!-- On-board IMU -->
     <link name="${ns}/oak_imu_frame"/>
-    <fixed_joint name="oak_imu_joint" parent="oak-d-base-frame" child="oak_imu_frame" xyz="0 0 0" rpy="0 0 0"/>
-    <!-- ============ VL53L5CX front ToF array (2026-09) ============
-         8x8 multizone ToF on a printed front bracket bolted to the chassis
-         front face. The bracket stands 24.5 mm proud of its mating face and
-         carries the breakout on a tab tilted 15 deg nose-down, so the array
-         looks forward and 15 deg down: it sees the floor and the low
-         obstacles that sit under the 0.340 m lidar plane.
-         Geometry from cad/VL53L5CX_test_assembly.STEP. That assembly holds
-         only the bracket and the breakout (no chassis), so the bracket-to-sensor
-         transform below is exact CAD, while tof_mount_joint is fitted to the
-         measured aperture height of 63.5 mm above the floor. Re-measure and
-         adjust tof_mount_joint's xyz if the bracket moves. Fitted against
-         base_joint 0.0815 (bottom plate caliper-measured 27.5 mm above the
-         floor, 2026-09-13); change both together.
-         tof_mount_link is the bracket's own CAD frame (+Z out the front,
-         +Y up, +X to the robot's left); the joint does the axis remap. -->
+    <xacro:fixed_joint name="oak_imu_joint" parent="oak-d-base-frame" child="oak_imu_frame" xyz="0 0 0" rpy="0 0 0"/>
+    <!-- ============ Dual VL53L5CX front ToF arrays (2026-09-19) ============
+         Source: stls/VL53LCX_mount.STEP. Upper adapter 15 deg, lower 40 deg.
+         Meshes are tessellated in CAD part frames, METRES (no 0.001 scale).
+         Mount CAD axes: +X robot-left, +Y up, +Z forward.
+         Starting attachment uses the old bracket's height/lateral origin.
+         Rear mating face moved from CAD z=-24.5 to -21.5 mm, so mount x
+         shifts back 3 mm to preserve that face's chassis position.
+         Refine ONLY tof_mount_joint for whole-assembly placement in RViz.
+         Sensor/adapter relative placements come from the STEP assembly.
+         Sensing origin uses the existing package-face point in board CAD:
+         (0, 2.45, -1.97) mm. Re-measure installed poses before perception use.
+         These are fixed adapter settings, not actuated joints.
+         Legacy tof_link aliases the upper sensor; dual Teensy ingestion and
+         downstream geometry configuration still require a separate update. -->
     <link name="${ns}/tof_mount_link">
-        <inertial>
-            <origin xyz="0 0.005 -0.005" rpy="0 0 0"/>
-            <mass value="0.030"/>
-            <inertia ixx="1.0E-05" ixy="0" ixz="0" iyy="1.5E-05" iyz="0" izz="1.0E-05"/>
-        </inertial>
-        <visual>
-            <origin xyz="0 0 0" rpy="0 0 0"/>
-            <geometry>
-                <mesh filename="package://yahboomcar_description/meshes/VL53L5CX_alt_front_mount.STL" scale="0.001 0.001 0.001"/>
-            </geometry>
-            <material name="White"/>
-        </visual>
-        <collision>
-            <origin xyz="0 0 0" rpy="0 0 0"/>
-            <geometry>
-                <mesh filename="package://yahboomcar_description/meshes/VL53L5CX_alt_front_mount.STL" scale="0.001 0.001 0.001"/>
-            </geometry>
-        </collision>
-        <!-- Breakout board. SolidWorks exported this STL translated into
-             positive space, so the visual origin carries the CAD part origin
-             back to (0,0,0) before the assembly transform is applied. -->
-        <visual>
-            <origin xyz="-0.012433 0.023431 0.020028" rpy="-2.8797982 -0.0016335 0.0060965"/>
-            <geometry>
-                <mesh filename="package://yahboomcar_description/meshes/VL53L5CX_sensor.STL" scale="0.001 0.001 0.001"/>
-            </geometry>
-            <material name="Green"/>
-        </visual>
-    </link>
-    <fixed_joint name="tof_mount_joint" parent="base_link" child="tof_mount_link" xyz="0.1320 0.0 -0.033549" rpy="1.5707963 0 1.5707963"/>
-    <!-- Sensing frame at the VL53L5CX package face, REP-103: +X is the
-         optical axis (forward, 15 deg down), +Z up. -->
+        <visual><origin xyz="0 0 0" rpy="0 0 0"/>
+            <geometry><mesh filename="package://yahboomcar_description/meshes/tof_dual_bracket.stl"/></geometry><material name=""><color rgba="0.75 0.75 0.78 1"/></material>
+        </visual>
+        <collision><origin xyz="0 0 0" rpy="0 0 0"/><geometry><mesh filename="package://yahboomcar_description/meshes/tof_dual_bracket.stl"/></geometry></collision>
+        <visual><origin xyz="0.000000000 0.114000000 0.003500000" rpy="0.000000000 -0.000000000 0.000000000"/>
+            <geometry><mesh filename="package://yahboomcar_description/meshes/tof_adapter_15.stl"/></geometry><material name=""><color rgba="0.75 0.75 0.78 1"/></material>
+        </visual>
+        <collision><origin xyz="0.000000000 0.114000000 0.003500000" rpy="0.000000000 -0.000000000 0.000000000"/><geometry><mesh filename="package://yahboomcar_description/meshes/tof_adapter_15.stl"/></geometry></collision>
+        <visual><origin xyz="0.000000000 0.020000000 0.003500000" rpy="0.000000000 -0.000000000 0.000000000"/>
+            <geometry><mesh filename="package://yahboomcar_description/meshes/tof_adapter_40.stl"/></geometry><material name=""><color rgba="0.75 0.75 0.78 1"/></material>
+        </visual>
+        <collision><origin xyz="0.000000000 0.020000000 0.003500000" rpy="0.000000000 -0.000000000 0.000000000"/><geometry><mesh filename="package://yahboomcar_description/meshes/tof_adapter_40.stl"/></geometry></collision>
+    </link>
+    <joint name="${ns}/tof_mount_joint" type="fixed">
+        <parent link="${ns}/base_link"/><child link="${ns}/tof_mount_link"/>
+        <origin xyz="0.1450 0.0 -0.030549" rpy="1.570796326795 0 1.570796326795"/>
+    </joint>
+    <link name="${ns}/tof_upper_board_link">
+        <visual><origin xyz="0 0 0" rpy="0 0 0"/>
+            <geometry><mesh filename="package://yahboomcar_description/meshes/tof_breakout.stl"/></geometry><material name=""><color rgba="0.05 0.35 0.12 1"/></material>
+        </visual>
+        <collision><origin xyz="0 0 0" rpy="0 0 0"/><geometry><mesh filename="package://yahboomcar_description/meshes/tof_breakout.stl"/></geometry></collision>
+    </link>
+    <joint name="${ns}/tof_upper_board_joint" type="fixed">
+        <parent link="${ns}/tof_mount_link"/><child link="${ns}/tof_upper_board_link"/>
+        <origin xyz="-0.000100000 0.113745168 0.016700834" rpy="-2.879793264 -0.000000000 0.000000000"/>
+    </joint>
+    <link name="${ns}/tof_upper_link"/>
+    <joint name="${ns}/tof_upper_joint" type="fixed">
+        <parent link="${ns}/tof_mount_link"/><child link="${ns}/tof_upper_link"/>
+        <origin xyz="-0.000100000 0.110868776 0.017969601" rpy="0.000000000 -1.308996939 -1.570796327"/>
+    </joint>
+    <link name="${ns}/tof_upper_optical_frame"/>
+    <joint name="${ns}/tof_upper_optical_joint" type="fixed">
+        <parent link="${ns}/tof_upper_link"/><child link="${ns}/tof_upper_optical_frame"/>
+        <origin xyz="0 0 0" rpy="-1.570796326795 0 -1.570796326795"/>
+    </joint>
+    <link name="${ns}/tof_lower_board_link">
+        <visual><origin xyz="0 0 0" rpy="0 0 0"/>
+            <geometry><mesh filename="package://yahboomcar_description/meshes/tof_breakout.stl"/></geometry><material name=""><color rgba="0.05 0.35 0.12 1"/></material>
+        </visual>
+        <collision><origin xyz="0 0 0" rpy="0 0 0"/><geometry><mesh filename="package://yahboomcar_description/meshes/tof_breakout.stl"/></geometry></collision>
+    </link>
+    <joint name="${ns}/tof_lower_board_joint" type="fixed">
+        <parent link="${ns}/tof_mount_link"/><child link="${ns}/tof_lower_board_link"/>
+        <origin xyz="-0.000100000 0.018035352 0.019528620" rpy="-2.443460930 -0.000000000 -0.000000000"/>
+    </joint>
+    <link name="${ns}/tof_lower_link"/>
+    <joint name="${ns}/tof_lower_joint" type="fixed">
+        <parent link="${ns}/tof_mount_link"/><child link="${ns}/tof_lower_link"/>
+        <origin xyz="-0.000100000 0.014892252 0.019462898" rpy="0.000000000 -0.872664626 -1.570796327"/>
+    </joint>
+    <link name="${ns}/tof_lower_optical_frame"/>
+    <joint name="${ns}/tof_lower_optical_joint" type="fixed">
+        <parent link="${ns}/tof_lower_link"/><child link="${ns}/tof_lower_optical_frame"/>
+        <origin xyz="0 0 0" rpy="-1.570796326795 0 -1.570796326795"/>
+    </joint>
     <link name="${ns}/tof_link"/>
-    <fixed_joint name="tof_joint" parent="tof_mount_link" child="tof_link" xyz="0.000115 0.016049 0.017941" rpy="0 -1.3089969 -1.5707963"/>
-    <!-- Optical convention (+Z along the optical axis, +X right, +Y down) -->
+    <joint name="${ns}/tof_joint" type="fixed">
+        <parent link="${ns}/tof_upper_link"/><child link="${ns}/tof_link"/>
+        <origin xyz="0 0 0" rpy="0 0 0"/>
+    </joint>
     <link name="${ns}/tof_optical_frame"/>
-    <fixed_joint name="tof_optical_joint" parent="tof_link" child="tof_optical_frame" xyz="0 0 0" rpy="-1.5707963 0 -1.5707963"/>
+    <joint name="${ns}/tof_optical_joint" type="fixed">
+        <parent link="${ns}/tof_link"/><child link="${ns}/tof_optical_frame"/>
+        <origin xyz="0 0 0" rpy="-1.570796326795 0 -1.570796326795"/>
+    </joint>
     <!-- ============ PAA5100JE optical flow sensor (2026-09-16) ============
          Downward-looking flow sensor that sits in a cut-out of a modified X3
@@ -346,9 +375,9 @@
         </visual>
     </link>
-    <fixed_joint name="paa5100je_plate_joint" parent="base_link" child="paa5100je_plate_link" xyz="-0.0344 0.0 -0.054" rpy="1.5707963 0 1.5707963"/>
+    <xacro:fixed_joint name="paa5100je_plate_joint" parent="base_link" child="paa5100je_plate_link" xyz="-0.0344 0.0 -0.054" rpy="1.5707963 0 1.5707963"/>
     <!-- Sensing frame at the centre of the lens face, axes aligned with
          base_link (+X forward, +Z up; the lens looks -Z). Its z in
          base_footprint is the sensor's height above the floor. -->
     <link name="${ns}/paa5100je_link"/>
-    <fixed_joint name="paa5100je_joint" parent="paa5100je_plate_link" child="paa5100je_link" xyz="-0.0005 -0.001 0.021" rpy="-1.5707963 -1.5707963 0"/>
+    <xacro:fixed_joint name="paa5100je_joint" parent="paa5100je_plate_link" child="paa5100je_link" xyz="-0.0005 -0.001 0.021" rpy="-1.5707963 -1.5707963 0"/>
 </robot>
