Commit message: fix(urdf): measure the lidar's X offset instead of assuming it
laser_joint x was -0.0115, recording a "55 mm rear" shift from the stock +0.0435.
Measured on the robot, that shift does not match reality.

Method: spin in place through five full turns capturing scans plus odom heading.
If the URDF offset is wrong by e, scan-to-map matching returns not the true
position but T_true + R(theta).e — so the estimated position traces a circle of
radius |e|. That is linear in (x_true, y_true, ex, ey), so it solves by least
squares with no curve fitting or local minima. The solver was validated first on
synthetic data: it recovers known offsets of 0, 8, 12 and 35 cm exactly, and to
within 6 mm under 2 cm of position noise.

Result over 101 scans spanning 1787 deg:
  ex = +0.056 +/- 0.007 m  (8.2 sigma)
  ey = -0.011 m, NOT significant (1.6 sigma)

ey being consistent with zero is the correct physical answer — the unit is
laterally centred — and doubles as a control, since a spurious fit would put mass
there too. Interleaved subsets agree to 1 mm. First vs second half disagree
(+0.031 vs +0.071), which is the 5 cm of drift during the spin leaking into the
fit, so the honest accuracy is +5..7 cm with ~3 cm systematic, not the +/-0.7 cm
statistical figure. Set to the central estimate, 0.055.

This brackets the stock X3 value (+0.0435), further evidence the rear-shift edit
was wrong. Chose the measurement over the stock figure because this chassis is an
X3 PLUS running the X3 description, so no stock dimension can be assumed to apply
— credit to the user for flagging that mismatch, which prompted this check.

A wrong value here is a lever arm: the scan swings about the wrong point as the
robot turns, and slam_toolbox bakes the same error into any map it builds. The
existing apartment map carries this distortion and MUST be rebuilt.

Co-Authored-By: Claude Opus 5 <noreply@anthropic.com>

File: src/yahboomcar_description/urdf/yahboomcar_X3.urdf (robot description, URDF)
Before this commit: robot yahboomcar, 18 links, 17 joints
Joints:
- joint laser_joint: origin xyz=-0.0115 5.25826986680105E-05 0.191 rpy=0 0 3.14159265 -> xyz=0.055 5.25826986680105E-05 0.191 rpy=0 0 3.14159265

Commit message: feat(description): tilting 2D->3D lidar mount with a revolute tilt joint
The lidar now rides in a carousel cradle that pitches forward/back in four
608RS bearings, driven by an LX-16A bus servo. Sweeping the tilt while the
2-D scanner spins is what produces the 3-D point cloud.

  base_link -> lidar_mount_link          plate + adapter + bracket + servo
            -> lidar_tilt_joint          revolute, axis +Y, positive = nose down
            -> lidar_tilt_link           carousel + coupler
            -> laser_link

Geometry is derived from cad/Prototype_Assembly.STEP, not eyeballed: the tilt
axis sits 153.0 mm above the mount base datum and 12.5 mm behind the lidar
centerline, and the lidar seat is 22.0 mm radially out from that axis, so
tilt=0 reproduces the previous flat scan plane. Masses and inertia tensors are
integrated over the actual meshes.

laser_link at tilt=0 is base_link (-0.0233, ~0, 0.2635). Note the CAD's 175 mm
internal rise and the measured lidar height do not fully reconcile: 17.5 mm of
gap remains between the bottom plate and the chassis deck. lidar_mount_joint's
z is the single number to trim if a better measurement turns up.

The display and its mount were removed from the robot to clear space, so
base_link now uses base_link_X3_noscreen.STL: the stock chassis mesh minus
every connected component reaching above z=0.075 (2340 of 69192 triangles).
base_link's inertial is still the stock 0.486 kg and has NOT been reduced.

Nothing publishes lidar_tilt_joint yet. joint_state_publisher already runs
headless in x3_bringup/x3_slam and will hold it at 0, which reproduces the old
fixed-lidar TF exactly; the real servo angle has to reach /joint_states before
an assembled 3-D cloud means anything.

Co-Authored-By: Claude Opus 5 (1M context) <noreply@anthropic.com>

File: src/yahboomcar_description/urdf/yahboomcar_X3.urdf (robot description, URDF)
Before this commit: robot yahboomcar, 18 links, 17 joints
Links:
- added link lidar_tilt_link, mass 0.0224; collision mesh filename=package://yahboomcar_description/meshes/4ros_carouselV3.STL scale=0.001 0.001 0.001; visual mesh filename=package://yahboomcar_description/meshes/4ros_carouselV3.STL scale=0.001 0.001 0.001
- link base_link: geometry collision mesh filename=package://yahboomcar_description/meshes/base_link_X3_noscre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; visual mesh filename=package://yahboomcar_description/meshes/base_link_X3_noscre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
- link lidar_mount_link: mass 0.035 -> 0.2387; geometry collision box size=0.0247 0.0381 0.0452; collision mesh filename=package://yahboomcar_description/meshes/4ROS_mount_adapterV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 scale=0.001 0.001 0.001
Joints:
- added joint lidar_tilt_joint: type revolute, parent lidar_mount_link, child lidar_tilt_link, origin xyz=-0.0125 0 0.153 rpy=0 0 0, axis 0 1 0, limit lower=-2.0944 upper=2.0944 effort=1.6 velocity=6.5
- joint laser_joint: origin xyz=-0.0115 5.25826986680105E-05 0.191 rpy=0 0 3.14159265 -> xyz=0 0 0.022 rpy=0 0 3.14159265; parent base_link -> lidar_tilt_link
- joint lidar_mount_joint: origin xyz=-0.0115 5.25826986680105E-05 0.116 rpy=0 0 0 -> xyz=-0.0108 5.25826986680105E-05 0.0885 rpy=0 0 0

File: src/yahboomcar_description/urdf/yahboomcar_X3.urdf.xacro (robot description, xacro)
@@ -110,28 +110,92 @@
         </inertial>
     </common_link>
+    <!-- ============ 2D->3D tilting lidar mount (2026-08) ============
+         Bottom plate + 4ROS adapter bolt to the chassis; the lidar rides in a
+         carousel cradle pitching in four 608RS bearings, driven by an LX-16A
+         bus servo. Geometry from yahboomcar_description/cad/Prototype_Assembly.STEP.
+         See yahboomcar_X3.urdf for the full derivation notes. -->
     <link name="${ns}/lidar_mount_link">
         <inertial>
-            <origin xyz="0 0 0.0375" rpy="0 0 0"/>
-            <mass value="0.035"/>
-            <inertia ixx="2.55E-05" ixy="0" ixz="0"
-                     iyy="2.55E-05" iyz="0" izz="1.76E-05"/>
-        </inertial>
+            <origin xyz="-0.01270 -0.02147 0.10269" rpy="0 0 0"/>
+            <mass value="0.2387"/>
+            <inertia ixx="1.1115E-03" ixy="1.0498E-06" ixz="-4.3702E-06"
+                     iyy="7.1579E-04" iyz="1.6225E-04" izz="4.7960E-04"/>
+        </inertial>
+        <xacro:macro name="mount_part" params="file xyz rpy">
+            <visual>
+                <origin xyz="${xyz}" rpy="${rpy}"/>
+                <geometry>
+                    <mesh filename="package://yahboomcar_description/meshes/${file}" scale="0.001 0.001 0.001"/>
+                </geometry>
+                <material name="White"/>
+            </visual>
+            <collision>
+                <origin xyz="${xyz}" rpy="${rpy}"/>
+                <geometry>
+                    <mesh filename="package://yahboomcar_description/meshes/${file}" scale="0.001 0.001 0.001"/>
+                </geometry>
+            </collision>
+        </xacro:macro>
+        <xacro:mount_part file="4ROS_mount_adapterV2.STL" xyz="0.035000 0.042000 0.000000" rpy="1.5707963 0 -1.5707963"/>
+        <xacro:mount_part file="bottomPlate.STL"          xyz="0.035000 0.042040 0.012000" rpy="1.5707963 0 -1.5707963"/>
+        <xacro:mount_part file="lx16_mountV2.STL"         xyz="0.002850 -0.039300 0.087875" rpy="1.5707963 0 -1.5707963"/>
+        <!-- LX-16A body: STEP only, drawn as its bounding box -->
         <visual>
-            <origin xyz="-0.0275 0.03368 0" rpy="1.5707963 0 0"/>
-            <geometry>
-                <mesh filename="package://yahboomcar_description/meshes/4ROS_lidar_mount.STL" scale="0.001 0.001 0.001"/>
+            <origin xyz="-0.012500 -0.075150 0.140650" rpy="0 0 0"/>
+            <geometry>
+                <box size="0.0247 0.0381 0.0452"/>
             </geometry>
             <material name="White"/>
         </visual>
         <collision>
-            <origin xyz="-0.0275 0.03368 0" rpy="1.5707963 0 0"/>
-            <geometry>
-                <mesh filename="package://yahboomcar_description/meshes/4ROS_lidar_mount.STL" scale="0.001 0.001 0.001"/>
+            <origin xyz="-0.012500 -0.075150 0.140650" rpy="0 0 0"/>
+            <geometry>
+                <box size="0.0247 0.0381 0.0452"/>
             </geometry>
         </collision>
+        <!-- 4x 608RS on the tilt axis; the pitch term is CAD clocking only -->
+        <xacro:macro name="mount_bearing" params="xyz rpy">
+            <visual>
+                <origin xyz="${xyz}" rpy="${rpy}"/>
+                <geometry>
+                    <mesh filename="package://yahboomcar_description/meshes/608RS.STL" scale="0.001 0.001 0.001"/>
+                </geometry>
+                <material name="White"/>
+            </visual>
+        </xacro:macro>
+        <xacro:mount_bearing xyz="0.003056 0.034900 0.153076"  rpy="1.5707963 0.7902475 -3.1415927"/>
+        <xacro:mount_bearing xyz="-0.027746 0.031300 0.149906" rpy="1.5707963 0.5851783 0"/>
+        <xacro:mount_bearing xyz="-0.023842 -0.024300 0.142353" rpy="1.5707963 0.0315727 0"/>
+        <xacro:mount_bearing xyz="-0.026141 -0.034900 0.145522" rpy="1.5707963 0.2839484 0"/>
     </link>
-    <!-- lidar moved 55 mm rearward, 6 mm up (2026); OAK-D took its old front spot -->
-    <fixed_joint name="lidar_mount_joint" parent="base_link" child="lidar_mount_link" xyz="-0.0115 5.25826986680105E-05 0.116" rpy="0 0 0"/>
-    <fixed_joint name="laser_joint" parent="base_link" child="laser_link" xyz="-0.0115 5.25826986680105E-05 0.191" rpy="0 0 3.14159265"/>
+    <fixed_joint name="lidar_mount_joint" parent="base_link" child="lidar_mount_link" xyz="-0.0108 5.25826986680105E-05 0.0885" rpy="0 0 0"/>
+    <!-- Rotating cradle: carousel + shaft coupler -->
+    <link name="${ns}/lidar_tilt_link">
+        <inertial>
+            <origin xyz="-0.00006 -0.01407 0.01659" rpy="0 0 0"/>
+            <mass value="0.0224"/>
+            <inertia ixx="1.729E-05" ixy="4.846E-08" ixz="-1.519E-08"
+                     iyy="6.351E-06" iyz="-6.114E-07" izz="2.068E-05"/>
+        </inertial>
+        <xacro:mount_part file="4ros_carouselV3.STL" xyz="0.030000 0.045049 -0.010000" rpy="1.5707963 0 -1.5707963"/>
+        <visual>
+            <origin xyz="0.004714 -0.024000 0.004714" rpy="-1.5707963 0 -3.1415927"/>
+            <geometry>
+                <mesh filename="package://yahboomcar_description/meshes/couplerV4.STL" scale="0.001 0.001 0.001"/>
+            </geometry>
+            <material name="White"/>
+        </visual>
+    </link>
+    <!-- axis +Y: positive noses the lidar DOWN. Limits are the LX-16A's own
+         +/-120 deg travel; nothing publishes this joint yet, so
+         joint_state_publisher holds it at 0 (= the old fixed-lidar TF). -->
+    <joint name="${ns}/lidar_tilt_joint" type="revolute">
+        <parent link="${ns}/lidar_mount_link"/>
+        <child link="${ns}/lidar_tilt_link"/>
+        <origin xyz="-0.0125 0 0.153" rpy="0 0 0"/>
+        <axis xyz="0 1 0"/>
+        <limit lower="-2.0944" upper="2.0944" effort="1.6" velocity="6.5"/>
+    </joint>
+    <fixed_joint name="laser_joint" parent="lidar_tilt_link" child="laser_link" xyz="0 0 0.022" rpy="0 0 3.14159265"/>
     <common_link name="camera_link" material="White" path="sensor">
         <inertial>

Commit message: fix(description): anchor the tilting mount on the MEASURED lidar x, not the stale one
The mount was placed by applying the new lidar's "11.8 mm rearward" offset to
laser_joint x = -0.0115. That baseline is wrong, and the robot's own working
tree has said so since 2026-08-08: x was measured on the robot as +0.055 by
spinning in place through 5 full turns and least-squares fitting the radius of
the circle the scan-to-map position traces when the offset is off. The -0.0115
recorded a "55 mm rear" shift that never happened.

Applying -11.8 mm to the measurement instead gives x = +0.0432, so
lidar_mount_joint x goes -0.0108 -> 0.0557. That is a 78 mm correction to the
lidar's position, which would otherwise have fed straight into SLAM and AMCL as
a lever arm error.

The measurement's derivation is carried into the URDF comment so it does not
get lost again, including the ey control (-0.011 m, 1.6 sigma, correctly not
significant) and the warning to remap after changing this value.

Co-Authored-By: Claude Opus 5 (1M context) <noreply@anthropic.com>

File: src/yahboomcar_description/urdf/yahboomcar_X3.urdf (robot description, URDF)
Before this commit: robot yahboomcar, 19 links, 18 joints
Joints:
- joint lidar_mount_joint: origin xyz=-0.0108 5.25826986680105E-05 0.0885 rpy=0 0 0 -> xyz=0.0557 5.25826986680105E-05 0.0885 rpy=0 0 0

File: src/yahboomcar_description/urdf/yahboomcar_X3.urdf.xacro (robot description, xacro)
@@ -169,5 +169,5 @@
         <xacro:mount_bearing xyz="-0.026141 -0.034900 0.145522" rpy="1.5707963 0.2839484 0"/>
     </link>
-    <fixed_joint name="lidar_mount_joint" parent="base_link" child="lidar_mount_link" xyz="-0.0108 5.25826986680105E-05 0.0885" rpy="0 0 0"/>
+    <fixed_joint name="lidar_mount_joint" parent="base_link" child="lidar_mount_link" xyz="0.0557 5.25826986680105E-05 0.0885" rpy="0 0 0"/>
     <!-- Rotating cradle: carousel + shaft coupler -->
     <link name="${ns}/lidar_tilt_link">

Commit message: feat(imu): replace the 10 Hz MPU9250 with an ICM-42688-P at 200 Hz
The old IMU was not slow because of the sensor. It reaches ROS through the
Rosmaster's 115200-baud serial bridge, sampled on Mcnamu_driver_X3's 0.1 s
pub_data timer alongside battery, version and joint states. That timer, not
the part, is the 10 Hz ceiling. Reading an ICM-42688-P directly off i2c-7
gives 200 Hz with Jetson-side timestamps instead of serial-arrival times.

Measured A/B with both IMUs publishing at once (src/imu_ab_compare.py):

    rate       10.1  ->  200.0 Hz   (19.9x)
    yaw bias  -6.84  ->   +1.04 deg/min
    |a|        9.828 ->    9.796    (expect 9.807)

Over 30 minutes parked that is -205 deg of phantom rotation down to +31 --
the drift that was bending the costmaps. Per-sample gyro noise is unchanged;
the MPU9250 is filtered internally before the serial hop, so sd is not a fair
comparison, and the real win is ~4.5x noise density from 20x the samples.

Mount orientation was MEASURED, not taken from the description: gravity sits
on sensor Z, so Z is up, not forward as assumed. A nose-up tilt drove sensor Y
to -2.96 m/s^2 and integrated -17.8 deg on sensor X; a left yaw gave sensor Z
+105.9 deg. Accel-derived tilt (17.2 deg) and gyro-integrated tilt (17.8 deg)
agree to 0.6 deg, cross-validating both axes and scale. The result is a pure
+90 deg yaw: ros_x=-sensor_y, ros_y=+sensor_x, ros_z=+sensor_z. Yaw needs NO
sign flip, so the -gz negation the upside-down MPU9250 requires is not carried
over.

The remap is applied in the node, not the URDF, because imu_filter_madgwick
does not consult TF; icm_imu_link is therefore deliberately identity rotation
and must stay that way or the rotation applies twice.

Three traps fixed along the way:

- imu_filter_param.yaml was keyed to `complementary_filter_gain_node` while
  the launch starts imu_filter_madgwick_node, so ROS 2 matched nothing and
  every value in it was silently ignored. Verified live: the node reported
  gain=0.1 (the built-in default) and use_mag=True while the file said
  otherwise. A wrong node-name key produces no warning at all.

- use_mag must be false. The ICM-42688-P is 6-axis with no magnetometer, and
  /imu/mag only ever came from the MPU9250. Gating the old IMU with use_mag
  true makes madgwick block forever, /imu/data stop, and the EKF silently lose
  its only IMU input.

- publish_imu gates ONLY imu/data_raw and imu/mag. The MPU9250 gyro is also
  the angular-velocity source for /vel_raw, because the firmware's own value
  is wrong (M2/M3 encoder cables are swapped). Gating that too breaks odom.

ekf_x3.yaml frequency 30 -> 50; at 30 the filter outran its own IMU input.

Verified live after relaunch: /imu/data_raw 200.7 Hz, /imu/data 199.6 Hz,
/odom 38.2 Hz, /vel_raw still 10 Hz, /scan 7.1 Hz, use_mag False, /imu/mag
gone, odom->base_footprint TF publishing, and the robot drives.

Co-Authored-By: Claude Opus 5 (1M context) <noreply@anthropic.com>

File: src/yahboomcar_description/urdf/yahboomcar_X3.urdf (robot description, URDF)
Before this commit: robot yahboomcar, 19 links, 18 joints
Links:
- added link icm_imu_link
Joints:
- added joint base_icm_imu: type fixed, parent base_link, child icm_imu_link, origin xyz=-0.03 0 0.0885 rpy=0 0 0

Commit message: feat(urdf): add the VL53L5CX front ToF array and its printed bracket
The 8x8 multizone ToF now has frames in the model, so it can be placed in
the costmap once it is wired: tof_mount_link (bracket), tof_link (REP-103,
+X along the optical axis) and tof_optical_frame.

The bracket->sensor transform is exact CAD, lifted from the placements in
VL53L5CX_test_assembly.STEP. The bracket had no STL in the repo, only STEP,
so meshes/VL53L5CX_alt_front_mount.STL is a tessellation of it.

Two facts worth keeping:

  - The VL53L5CX package sits on the -Z face of the breakout, not the +Z
    face the pin header protrudes from. That is what fixes the mount's
    orientation on the robot: the optical axis comes out of the tab
    forward and 15 deg down, which is the only orientation that makes
    sense for a sensor meant to see the floor and the obstacles below the
    0.340 m lidar plane.

  - tof_mount_joint is not from CAD. The assembly holds only the bracket
    and the breakout, no chassis, so the pose on base_link was fitted to
    the measured aperture height (64.0 mm above the floor) and then
    trimmed against the rendered model. Re-measure if the bracket moves.

The aperture lands at x=0.1499 m, 0.0640 m above the floor; the optical
axis meets the floor about 0.39 m ahead.

Note the two description files disagree on base_joint (0.076 vs 0.0815),
which predates this change; the joint xyz here is base_link-relative in
both, so the heights above quote the plain .urdf that the robot loads.

Co-Authored-By: Claude Opus 5 (1M context) <noreply@anthropic.com>

File: src/yahboomcar_description/urdf/yahboomcar_X3.urdf (robot description, URDF)
Before this commit: robot yahboomcar, 21 links, 20 joints
Links:
- added link tof_link
- added link tof_mount_link, mass 0.030; collision mesh filename=package://yahboomcar_description/meshes/VL53L5CX_alt_front_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 scale=0.001 0.001 0.001; visual mesh filename=package://yahboomcar_description/meshes/VL53L5CX_alt_front_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 scale=0.001 0.001 0.001
- added link tof_optical_frame
Joints:
- added joint tof_joint: type fixed, parent tof_mount_link, child tof_link, origin xyz=0.000115 0.016049 0.017941 rpy=0 -1.3089969 -1.5707963
- added joint tof_mount_joint: type fixed, parent base_link, child tof_mount_link, origin xyz=0.1320 0.0 -0.028049 rpy=1.5707963 0 1.5707963
- added joint tof_optical_joint: type fixed, parent tof_link, child tof_optical_frame, origin xyz=0 0 0 rpy=-1.5707963 0 -1.5707963

File: src/yahboomcar_description/urdf/yahboomcar_X3.urdf.xacro (robot description, xacro)
@@ -250,3 +250,56 @@
     <link name="${ns}/oak_imu_frame"/>
     <fixed_joint name="oak_imu_joint" parent="oak-d-base-frame" child="oak_imu_frame" xyz="0 0 0" rpy="0 0 0"/>
+    <!-- ============ VL53L5CX front ToF array (2026-09) ============
+         8x8 multizone ToF on a printed front bracket bolted to the chassis
+         front face. The bracket stands 24.5 mm proud of its mating face and
+         carries the breakout on a tab tilted 15 deg nose-down, so the array
+         looks forward and 15 deg down: it sees the floor and the low
+         obstacles that sit under the 0.340 m lidar plane.
+         Geometry from cad/VL53L5CX_test_assembly.STEP. That assembly holds
+         only the bracket and the breakout (no chassis), so the bracket-to-sensor
+         transform below is exact CAD, while tof_mount_joint is fitted to the
+         measured aperture height of 63.5 mm above the floor. Re-measure and
+         adjust tof_mount_joint's xyz if the bracket moves. NOTE the two files
+         disagree on base_joint (0.076 here vs 0.0815 in the other), a
+         pre-existing 5.5 mm split; this xyz is base_link-relative in both.
+         tof_mount_link is the bracket's own CAD frame (+Z out the front,
+         +Y up, +X to the robot's left); the joint does the axis remap. -->
+    <link name="${ns}/tof_mount_link">
+        <inertial>
+            <origin xyz="0 0.005 -0.005" rpy="0 0 0"/>
+            <mass value="0.030"/>
+            <inertia ixx="1.0E-05" ixy="0" ixz="0" iyy="1.5E-05" iyz="0" izz="1.0E-05"/>
+        </inertial>
+        <visual>
+            <origin xyz="0 0 0" rpy="0 0 0"/>
+            <geometry>
+                <mesh filename="package://yahboomcar_description/meshes/VL53L5CX_alt_front_mount.STL" scale="0.001 0.001 0.001"/>
+            </geometry>
+            <material name="White"/>
+        </visual>
+        <collision>
+            <origin xyz="0 0 0" rpy="0 0 0"/>
+            <geometry>
+                <mesh filename="package://yahboomcar_description/meshes/VL53L5CX_alt_front_mount.STL" scale="0.001 0.001 0.001"/>
+            </geometry>
+        </collision>
+        <!-- Breakout board. SolidWorks exported this STL translated into
+             positive space, so the visual origin carries the CAD part origin
+             back to (0,0,0) before the assembly transform is applied. -->
+        <visual>
+            <origin xyz="-0.012433 0.023431 0.020028" rpy="-2.8797982 -0.0016335 0.0060965"/>
+            <geometry>
+                <mesh filename="package://yahboomcar_description/meshes/VL53L5CX_sensor.STL" scale="0.001 0.001 0.001"/>
+            </geometry>
+            <material name="Green"/>
+        </visual>
+    </link>
+    <fixed_joint name="tof_mount_joint" parent="base_link" child="tof_mount_link" xyz="0.1320 0.0 -0.028049" rpy="1.5707963 0 1.5707963"/>
+    <!-- Sensing frame at the VL53L5CX package face, REP-103: +X is the
+         optical axis (forward, 15 deg down), +Z up. -->
+    <link name="${ns}/tof_link"/>
+    <fixed_joint name="tof_joint" parent="tof_mount_link" child="tof_link" xyz="0.000115 0.016049 0.017941" rpy="0 -1.3089969 -1.5707963"/>
+    <!-- Optical convention (+Z along the optical axis, +X right, +Y down) -->
+    <link name="${ns}/tof_optical_frame"/>
+    <fixed_joint name="tof_optical_joint" parent="tof_link" child="tof_optical_frame" xyz="0 0 0" rpy="-1.5707963 0 -1.5707963"/>
 </robot>
