Commit message: feat(urdf): add the PAA5100JE flow sensor, fit base_joint to 0.0815 in both files
Adds the downward flow-sensor plate and breakout meshes plus the STEP/STL
sources in stls/, and moves the .urdf to the caliper-measured base_joint
(0.0815) the xacro already used, re-deriving the OAK and ToF z offsets.

Co-Authored-By: Claude Opus 5 (1M context) <noreply@anthropic.com>

File: src/yahboomcar_description/urdf/yahboomcar_X3.urdf (robot description, URDF)
Before this commit: robot yahboomcar, 24 links, 23 joints
Links:
- added link paa5100je_link
- added link paa5100je_mount_link, mass 0.130; collision mesh filename=package://yahboomcar_description/meshes/paa5100je_bottom_mo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 scale=0.001 0.001 0.001; visual mesh filename=package://yahboomcar_description/meshes/PAA5100JE_sensor.STL scale=0.001 0.001 0.001
Joints:
- added joint paa5100je_joint: type fixed, parent paa5100je_mount_link, child paa5100je_link, origin xyz=0 -0.011 0.029906 rpy=-1.5707963 -1.5707963 0
- added joint paa5100je_mount_joint: type fixed, parent base_link, child paa5100je_mount_link, origin xyz=-0.038 0.0 -0.060 rpy=1.5707963 0 1.5707963
- joint base_joint: origin xyz=0.0 0.0 0.076 rpy=0 0 0 -> xyz=0.0 0.0 0.0815 rpy=0 0 0
- joint oak_center_joint: origin xyz=0.107315 1.7948E-05 0.134 rpy=0 0 0 -> xyz=0.107315 1.7948E-05 0.1285 rpy=0 0 0
- joint tof_mount_joint: origin xyz=0.1320 0.0 -0.028049 rpy=1.5707963 0 1.5707963 -> xyz=0.1320 0.0 -0.033549 rpy=1.5707963 0 1.5707963

File: src/yahboomcar_description/urdf/yahboomcar_X3.urdf.xacro (robot description, xacro)
@@ -260,7 +260,7 @@
          transform below is exact CAD, while tof_mount_joint is fitted to the
          measured aperture height of 63.5 mm above the floor. Re-measure and
-         adjust tof_mount_joint's xyz if the bracket moves. NOTE the two files
-         disagree on base_joint (0.076 here vs 0.0815 in the other), a
-         pre-existing 5.5 mm split; this xyz is base_link-relative in both.
+         adjust tof_mount_joint's xyz if the bracket moves. Fitted against
+         base_joint 0.0815 (bottom plate caliper-measured 27.5 mm above the
+         floor, 2026-09-13); change both together.
          tof_mount_link is the bracket's own CAD frame (+Z out the front,
          +Y up, +X to the robot's left); the joint does the axis remap. -->
@@ -295,5 +295,5 @@
         </visual>
     </link>
-    <fixed_joint name="tof_mount_joint" parent="base_link" child="tof_mount_link" xyz="0.1320 0.0 -0.028049" rpy="1.5707963 0 1.5707963"/>
+    <fixed_joint name="tof_mount_joint" parent="base_link" child="tof_mount_link" xyz="0.1320 0.0 -0.033549" rpy="1.5707963 0 1.5707963"/>
     <!-- Sensing frame at the VL53L5CX package face, REP-103: +X is the
          optical axis (forward, 15 deg down), +Z up. -->
@@ -303,3 +303,46 @@
     <link name="${ns}/tof_optical_frame"/>
     <fixed_joint name="tof_optical_joint" parent="tof_link" child="tof_optical_frame" xyz="0 0 0" rpy="-1.5707963 0 -1.5707963"/>
+    <!-- ============ PAA5100JE optical flow sensor (2026-09) ============
+         Downward-looking flow sensor on a printed plate under the chassis
+         bottom edge. Geometry from stls/pa5100je_assembly.STEP, which holds
+         only the plate and the breakout: the plate-to-sensor transform below
+         is exact CAD (sensor at plate (0, -6, 29.906) mm, yawed 180 deg), while
+         paa5100je_mount_joint is a FIRST GUESS to be corrected in
+         `laptop_sim.sh view` against the real robot.
+         paa5100je_mount_link is the plate's CAD frame (+X across the robot,
+         +Y up away from the sensor, +Z along the robot's +X). Both STLs were
+         exported translated into positive space; the visual origins undo it. -->
+    <link name="${ns}/paa5100je_mount_link">
+        <inertial>
+            <origin xyz="0 0.002 0.040" rpy="0 0 0"/>
+            <mass value="0.130"/>
+            <inertia ixx="2.0E-04" ixy="0" ixz="0" iyy="5.0E-04" iyz="0" izz="3.0E-04"/>
+        </inertial>
+        <visual>
+            <origin xyz="-0.081 -0.006 -0.030" rpy="0 0 0"/>
+            <geometry>
+                <mesh filename="package://yahboomcar_description/meshes/paa5100je_bottom_mount.STL" scale="0.001 0.001 0.001"/>
+            </geometry>
+            <material name="White"/>
+        </visual>
+        <collision>
+            <origin xyz="-0.081 -0.006 -0.030" rpy="0 0 0"/>
+            <geometry>
+                <mesh filename="package://yahboomcar_description/meshes/paa5100je_bottom_mount.STL" scale="0.001 0.001 0.001"/>
+            </geometry>
+        </collision>
+        <visual>
+            <origin xyz="0.012 -0.006 0.017906" rpy="0 0 3.1415927"/>
+            <geometry>
+                <mesh filename="package://yahboomcar_description/meshes/PAA5100JE_sensor.STL" scale="0.001 0.001 0.001"/>
+            </geometry>
+            <material name="Green"/>
+        </visual>
+    </link>
+    <fixed_joint name="paa5100je_mount_joint" parent="base_link" child="paa5100je_mount_link" xyz="-0.038 0.0 -0.060" rpy="1.5707963 0 1.5707963"/>
+    <!-- Sensing frame at the centre of the breakout's floor-facing face,
+         axes aligned with base_link (+X forward, +Z up; the lens looks -Z).
+         Its z in base_footprint is the sensor's height above the floor. -->
+    <link name="${ns}/paa5100je_link"/>
+    <fixed_joint name="paa5100je_joint" parent="paa5100je_mount_link" child="paa5100je_link" xyz="0 -0.011 0.029906" rpy="-1.5707963 -1.5707963 0"/>
 </robot>

Commit message: feat(urdf): mount the PAA5100JE in a modified bottom plate
The first printed mount hung the flow sensor ~10 mm off the floor, well
below its ~15-35 mm working range. The redesign sets the sensor into a
cut-out in a modified X3 Plus bottom plate, with a printed mount on top.

Placement below the plate is exact CAD from paa5100je_assembly3.STEP; the
lens face sits 1 mm under the plate, 26.5 mm above the floor with
base_joint 0.0815. The plate's fore/aft position was set by eye in the
URDF viewer. Plate and mount meshes were converted from STEP in their
part frames.

Co-Authored-By: Claude Opus 5 (1M context) <noreply@anthropic.com>

File: src/yahboomcar_description/urdf/yahboomcar_X3.urdf (robot description, URDF)
Before this commit: robot yahboomcar, 26 links, 25 joints
Links:
- removed link paa5100je_mount_link
- added link paa5100je_plate_link, mass 0.150; visual mesh filename=package://yahboomcar_description/meshes/PAA5100JE_sensor.STL scale=0.001 0.001 0.001; visual mesh filename=package://yahboomcar_description/meshes/X3plus_bottom_plate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
Joints:
- removed joint paa5100je_mount_joint
- added joint paa5100je_plate_joint: type fixed, parent base_link, child paa5100je_plate_link, origin xyz=-0.0344 0.0 -0.054 rpy=1.5707963 0 1.5707963
- joint paa5100je_joint: origin xyz=0 -0.011 0.029906 rpy=-1.5707963 -1.5707963 0 -> xyz=-0.0005 -0.001 0.021 rpy=-1.5707963 -1.5707963 0; parent paa5100je_mount_link -> paa5100je_plate_link

File: src/yahboomcar_description/urdf/yahboomcar_X3.urdf.xacro (robot description, xacro)
@@ -303,35 +303,41 @@
     <link name="${ns}/tof_optical_frame"/>
     <fixed_joint name="tof_optical_joint" parent="tof_link" child="tof_optical_frame" xyz="0 0 0" rpy="-1.5707963 0 -1.5707963"/>
-    <!-- ============ PAA5100JE optical flow sensor (2026-09) ============
-         Downward-looking flow sensor on a printed plate under the chassis
-         bottom edge. Geometry from stls/pa5100je_assembly.STEP, which holds
-         only the plate and the breakout: the plate-to-sensor transform below
-         is exact CAD (sensor at plate (0, -6, 29.906) mm, yawed 180 deg), while
-         paa5100je_mount_joint is a FIRST GUESS to be corrected in
-         `laptop_sim.sh view` against the real robot.
-         paa5100je_mount_link is the plate's CAD frame (+X across the robot,
-         +Y up away from the sensor, +Z along the robot's +X). Both STLs were
-         exported translated into positive space; the visual origins undo it. -->
-    <link name="${ns}/paa5100je_mount_link">
-        <inertial>
-            <origin xyz="0 0.002 0.040" rpy="0 0 0"/>
-            <mass value="0.130"/>
-            <inertia ixx="2.0E-04" ixy="0" ixz="0" iyy="5.0E-04" iyz="0" izz="3.0E-04"/>
-        </inertial>
-        <visual>
-            <origin xyz="-0.081 -0.006 -0.030" rpy="0 0 0"/>
-            <geometry>
-                <mesh filename="package://yahboomcar_description/meshes/paa5100je_bottom_mount.STL" scale="0.001 0.001 0.001"/>
-            </geometry>
-            <material name="White"/>
-        </visual>
-        <collision>
-            <origin xyz="-0.081 -0.006 -0.030" rpy="0 0 0"/>
-            <geometry>
-                <mesh filename="package://yahboomcar_description/meshes/paa5100je_bottom_mount.STL" scale="0.001 0.001 0.001"/>
-            </geometry>
-        </collision>
-        <visual>
-            <origin xyz="0.012 -0.006 0.017906" rpy="0 0 3.1415927"/>
+    <!-- ============ PAA5100JE optical flow sensor (2026-09-16) ============
+         Downward-looking flow sensor that sits in a cut-out of a modified X3
+         Plus bottom plate, held by a printed mount on top of the plate.
+         Geometry from stls/paa5100je_assembly3.STEP, whose placements are all
+         relative to the plate, so everything below the plate joint is exact
+         CAD: mount at plate (-1, 14, 27.5) mm, sensor at (-0.5, 4, 21) mm
+         flipped 180 deg about X. The lens face ends up 1 mm below the plate
+         underside, i.e. ~26.5 mm above the floor with base_joint 0.0815.
+         paa5100je_plate_link is the plate's CAD frame: +X across the robot,
+         +Y up (y=0 is the underside), +Z along the robot's +X. Its joint puts
+         the underside on the chassis bottom (base_link z=-0.054); the fore/aft
+         x and which end faces forward are NOT verified against the robot.
+         The plate and mount STLs were converted from STEP in their part
+         frames (metres); the sensor STL is the SolidWorks export (mm,
+         translated into positive space, undone by its visual origin). -->
+    <link name="${ns}/paa5100je_plate_link">
+        <inertial>
+            <origin xyz="0 0.005 0" rpy="0 0 0"/>
+            <mass value="0.150"/>
+            <inertia ixx="5.5E-04" ixy="0" ixz="0" iyy="8.8E-04" iyz="0" izz="3.3E-04"/>
+        </inertial>
+        <visual>
+            <origin xyz="0 0 0" rpy="0 0 0"/>
+            <geometry>
+                <mesh filename="package://yahboomcar_description/meshes/X3plus_bottom_plate_modified.STL"/>
+            </geometry>
+            <material name="White"/>
+        </visual>
+        <visual>
+            <origin xyz="-0.001 0.014 0.0275" rpy="1.5707963 0 0"/>
+            <geometry>
+                <mesh filename="package://yahboomcar_description/meshes/paa5100je_left_centered_mount.STL"/>
+            </geometry>
+            <material name="White"/>
+        </visual>
+        <visual>
+            <origin xyz="-0.0125 0.004 0.033" rpy="3.1415927 0 0"/>
             <geometry>
                 <mesh filename="package://yahboomcar_description/meshes/PAA5100JE_sensor.STL" scale="0.001 0.001 0.001"/>
@@ -340,9 +346,9 @@
         </visual>
     </link>
-    <fixed_joint name="paa5100je_mount_joint" parent="base_link" child="paa5100je_mount_link" xyz="-0.038 0.0 -0.060" rpy="1.5707963 0 1.5707963"/>
-    <!-- Sensing frame at the centre of the breakout's floor-facing face,
-         axes aligned with base_link (+X forward, +Z up; the lens looks -Z).
-         Its z in base_footprint is the sensor's height above the floor. -->
+    <fixed_joint name="paa5100je_plate_joint" parent="base_link" child="paa5100je_plate_link" xyz="-0.0344 0.0 -0.054" rpy="1.5707963 0 1.5707963"/>
+    <!-- Sensing frame at the centre of the lens face, axes aligned with
+         base_link (+X forward, +Z up; the lens looks -Z). Its z in
+         base_footprint is the sensor's height above the floor. -->
     <link name="${ns}/paa5100je_link"/>
-    <fixed_joint name="paa5100je_joint" parent="paa5100je_mount_link" child="paa5100je_link" xyz="0 -0.011 0.029906" rpy="-1.5707963 -1.5707963 0"/>
+    <fixed_joint name="paa5100je_joint" parent="paa5100je_plate_link" child="paa5100je_link" xyz="-0.0005 -0.001 0.021" rpy="-1.5707963 -1.5707963 0"/>
 </robot>

Commit message: Replace the OAK-D Lite with the OAK-D Pro W in the URDF
The Pro W sits on a new printed bracket (stls/oakdpro_mount.STL). Its
body and bracket meshes are exported from stls/oakd_pro_assembly.STEP
into oak-d-base-frame, so the URDF uses them at zero offset.

oak_center_joint is fitted to the installed bracket in RViz: 0.5 mm
forward and 1.0 mm lower than the Lite, putting the optical centre
0.209 m above the floor. The driver's OAK_MOUNT_X/Z and the ground-plane
camera_height_m follow it. camera_pitch_deg is still the Lite's value
and needs re-measuring.

Co-Authored-By: Claude Opus 5.5 (1M context) <noreply@anthropic.com>

File: src/yahboomcar_description/urdf/yahboomcar_X3.urdf (robot description, URDF)
Before this commit: robot yahboomcar, 32 links, 31 joints
Links:
- link oak-d-base-frame: mass 0.0611 -> 0.15; geometry collision box size=0.0231 0.097 0.0295; visual mesh filename=package://yahboomcar_description/meshes/oakd_pro_w.stl
Joints:
- joint oak_center_joint: origin xyz=0.107315 1.7948E-05 0.1285 rpy=0 0 0 -> xyz=0.107815 1.7948E-05 0.1275 rpy=0 0 0

Commit message: Fix OAK-D Pro W stretched-preview intrinsics; set measured height
The CAM_A 480x640 grid is the 16:9 1080P ISP output stretched, so
getCameraIntrinsics' uniform scale gave fy ~285 instead of ~676 and a
wrong cy. Map the EEPROM K through the sensor's real 1080P crop
(IMX214 Lite and IMX378 Pro W) in the driver and floor validator.

Lens centre calipered at 0.213 m: URDF oak_center_joint z, OAK_MOUNT_Z
and camera_height_m move together. Pitch set to -1.044 deg from the one
clean floor fit (IMU agrees at -1.0); later fits were not repeatable.

The validator no longer assumes gravity on IMU +Y: the BNO086's down
axis is -X and its EEPROM IMU extrinsics are identity.

Co-Authored-By: Claude Opus 5.5 (1M context) <noreply@anthropic.com>

File: src/yahboomcar_description/urdf/yahboomcar_X3.urdf (robot description, URDF)
Before this commit: robot yahboomcar, 32 links, 31 joints
Joints:
- joint oak_center_joint: origin xyz=0.107815 1.7948E-05 0.1275 rpy=0 0 0 -> xyz=0.107815 1.7948E-05 0.1315 rpy=0 0 0

Commit message: URDF: lidar yaw 180 + 4.85 deg, the mount's measured error
laser_joint now carries the yaw measured by lidar_yaw_calib.py, so SLAM,
Nav2 and RViz place scans where the CBF already does. Maps saved before
this were built with the lidar at exactly 180 deg.

lidar_yaw_calib.py --use-tf places scans by the TF tree, to check the
corrected URDF end to end.

Co-Authored-By: Claude Opus 5.5 <noreply@anthropic.com>

File: src/yahboomcar_description/urdf/yahboomcar_X3.urdf (robot description, URDF)
Before this commit: robot yahboomcar, 32 links, 31 joints
Joints:
- joint laser_joint: origin xyz=0 0 0.022 rpy=0 0 3.14159265 -> xyz=0 0 0.022 rpy=0 0 3.226241

File: src/yahboomcar_description/urdf/yahboomcar_X3.urdf.xacro (robot description, xacro)
@@ -197,5 +197,5 @@
         <limit lower="-2.0944" upper="2.0944" effort="1.6" velocity="6.5"/>
     </joint>
-    <xacro:fixed_joint name="laser_joint" parent="lidar_tilt_link" child="laser_link" xyz="0 0 0.022" rpy="0 0 3.14159265"/>
+    <xacro:fixed_joint name="laser_joint" parent="lidar_tilt_link" child="laser_link" xyz="0 0 0.022" rpy="0 0 3.226241"/>  <!-- 180 + 4.85 deg measured mount yaw, see yahboomcar_X3.urdf -->
     <xacro:common_link name="camera_link" material="White" path="sensor">
         <inertial>

Commit message: Restore /scan from the Livox Mid-360S (livox_scan_node)
The YDLidar was replaced by the Livox, leaving /scan unpublished: the CBF
had only the bumper ToF and AMCL/SLAM had nothing. livox_scan_node slices
the cloud at z +-0.05 m around the sensor (0.26-0.36 m above the floor,
the old scan plane was 0.3185 m) into /scan and /scan_fixed, 720 beams,
in the old laser_link so server_x3, AMCL and the existing maps work
unchanged. Two-frame min merge (~96% of beams return), yaw de-skew from
/odom. CustomMsg is decoded from raw CDR bytes: rclpy's deserializer
takes 177 ms per 20k-point message on the Orin, the numpy view 0.3 ms.

URDF: lidar_tilt_joint is now fixed (nothing publishes it since the
servo was removed, which disconnected laser_link) and a provisional
livox_frame joint is added (height from livox_floor_fit, 0.31 m).
x3_bringup launches the Livox driver; server_x3 sources ~/ws_livox.

Tested 2026-10-29: CBF box stop works; auto pose on newApartment1
accepts at margin 2.7-3.4.

Co-Authored-By: Claude Opus 5.5 <noreply@anthropic.com>

File: src/yahboomcar_description/urdf/yahboomcar_X3.urdf (robot description, URDF)
Before this commit: robot yahboomcar, 32 links, 31 joints
Links:
- added link livox_frame
Joints:
- added joint livox_joint: type fixed, parent base_link, child livox_frame, origin xyz=0.0432 0 0.2285 rpy=0 0 0
- joint lidar_tilt_joint: axis 0 1 0 -> (none); limit lower=-2.0944 upper=2.0944 effort=1.6 velocity=6.5 -> (none); type revolute -> fixed
